File: BRK-SC-70-6/BRK-SC-70-6.kicad_pcb (KiCad board)
At the start: 2 copper layers, 18.3 x 18 mm, 3 parts, among them J1 Conn_01x03, J2 Conn_01x03, U1 Conn_02x03_Counter_Clockwise

Commit message: Minor updates
Other:
- rule solder_mask_min_width: 0.25 -> 0.2
Changed lines of the file:
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@@
     (pad_drill 0.762)
     (pad_to_mask_clearance 0)
-    (solder_mask_min_width 0.25)
+    (solder_mask_min_width 0.2)
     (aux_axis_origin 0 0)
     (visible_elements FFFFFF7F)
