File: BUS-BLASTER-AVR/BUS-BLASTER-AVR.kicad_pcb (KiCad board)
At the start: 2 copper layers, 54 x 37 mm, 6 parts, among them J1 Conn_02x05_Odd_Even, J2 Conn_02x10_Odd_Even

Commit message: Minor updates
Other:
- outline, holes or cut-outs redrawn
- rule pad_to_mask_clearance: 0.2 -> 0
Changed lines of the file:
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@@
-(kicad_pcb (version 20171130) (host pcbnew 5.0.1-33cea8e~68~ubuntu18.04.1)
+(kicad_pcb (version 20171130) (host pcbnew 5.0.1-33cea8e~68~ubuntu18.10.1)
   (general
     (thickness 1.6)
-    (drawings 27)
+    (drawings 31)
     (tracks 36)
     (zones 0)
@@
     (pad_size 1.524 1.524)
     (pad_drill 0.762)
-    (pad_to_mask_clearance 0.2)
+    (pad_to_mask_clearance 0)
     (solder_mask_min_width 0.2)
     (aux_axis_origin 0 0)
@@
     )
   )
+  (gr_arc (start 100 52) (end 102 52) (angle -90) (layer Edge.Cuts) (width 0.15))
+  (gr_arc (start 100 85) (end 100 87) (angle -90) (layer Edge.Cuts) (width 0.15))
+  (gr_arc (start 50 85) (end 48 85) (angle -90) (layer Edge.Cuts) (width 0.15))
+  (gr_arc (start 50 52) (end 50 50) (angle -90) (layer Edge.Cuts) (width 0.15))
   (gr_text "BUS-BLASTER-AVR v1.0\nhttps://gekkio.fi" (at 67.6 53.4) (layer F.SilkS)
     (effects (font (size 1.2 1.2) (thickness 0.3)))
@@
     (effects (font (size 1 1) (thickness 0.15)) (justify left))
   )
-  (gr_line (start 48 50) (end 102 50) (layer Edge.Cuts) (width 0.15))
-  (gr_line (start 102 87) (end 102 50) (layer Edge.Cuts) (width 0.15))
-  (gr_line (start 48 87) (end 102 87) (layer Edge.Cuts) (width 0.15))
-  (gr_line (start 48 50) (end 48 87) (layer Edge.Cuts) (width 0.15))
+  (gr_line (start 50 50) (end 100 50) (layer Edge.Cuts) (width 0.15))
+  (gr_line (start 102 85) (end 102 52) (layer Edge.Cuts) (width 0.15))
+  (gr_line (start 50 87) (end 100 87) (layer Edge.Cuts) (width 0.15))
+  (gr_line (start 48 52) (end 48 85) (layer Edge.Cuts) (width 0.15))
   (segment (start 83.1 67.26) (end 74.64 67.26) (width 0.6) (layer F.Cu) (net 5))
   (segment (start 74.64 67.26) (end 68.32 73.58) (width 0.6) (layer F.Cu) (net 5))
