File: PIC-ICSP-504050/PIC-ICSP-504050.kicad_pcb (KiCad board)
At the start: 2 copper layers, 30 x 40 mm, 6 parts, among them J1 Conn_01x05_MountingPin, J2 Conn_01x06

Commit message: Minor updates
Other:
- outline, holes or cut-outs redrawn
- rule pad_to_mask_clearance: 0.2 -> 0
Changed lines of the file:
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@@
-(kicad_pcb (version 20171130) (host pcbnew 5.0.1-33cea8e~68~ubuntu18.04.1)
+(kicad_pcb (version 20171130) (host pcbnew 5.0.1-33cea8e~68~ubuntu18.10.1)
   (general
     (thickness 1.6)
-    (drawings 11)
+    (drawings 15)
     (tracks 13)
     (zones 0)
@@
     (pad_size 1.524 1.524)
     (pad_drill 0.762)
-    (pad_to_mask_clearance 0.2)
+    (pad_to_mask_clearance 0)
     (solder_mask_min_width 0.2)
     (aux_axis_origin 0 0)
@@
     (pad 1 np_thru_hole circle (at 0 0) (size 3.2 3.2) (drill 3.2) (layers *.Cu *.Mask))
   )
+  (gr_arc (start 78 52) (end 80 52) (angle -90) (layer Edge.Cuts) (width 0.15))
+  (gr_arc (start 78 88) (end 78 90) (angle -90) (layer Edge.Cuts) (width 0.15))
+  (gr_arc (start 52 88) (end 50 88) (angle -90) (layer Edge.Cuts) (width 0.15))
+  (gr_arc (start 52 52) (end 52 50) (angle -90) (layer Edge.Cuts) (width 0.15))
   (gr_text "PIC-ICSP-504050 v1.0\nhttps://gekkio.fi" (at 65.15 80.45) (layer F.SilkS)
     (effects (font (size 1.2 1.2) (thickness 0.3)))
@@
     (effects (font (size 1.5 1.5) (thickness 0.3)) (justify left))
   )
-  (gr_line (start 50 90) (end 50 50) (layer Edge.Cuts) (width 0.15))
-  (gr_line (start 50 90) (end 80 90) (layer Edge.Cuts) (width 0.15))
-  (gr_line (start 80 50) (end 80 90) (layer Edge.Cuts) (width 0.15))
-  (gr_line (start 50 50) (end 80 50) (layer Edge.Cuts) (width 0.15))
+  (gr_line (start 50 88) (end 50 52) (layer Edge.Cuts) (width 0.15))
+  (gr_line (start 52 90) (end 78 90) (layer Edge.Cuts) (width 0.15))
+  (gr_line (start 80 52) (end 80 88) (layer Edge.Cuts) (width 0.15))
+  (gr_line (start 52 50) (end 78 50) (layer Edge.Cuts) (width 0.15))
   (segment (start 63.395 63.7) (end 69.45 63.7) (width 0.6) (layer F.Cu) (net 1))
   (segment (start 69.45 63.7) (end 70.9 63.7) (width 0.6) (layer F.Cu) (net 1))
