File: BRK-VSSOP-8-2.4x2.1-P0.5/BRK-VSSOP-8-2.4x2.1-P0.5.sch (KiCad schematic (older format))
At the start: 3 parts, among them J1 Conn_01x03, J2 Conn_01x03, U1 SC-70-6

Commit message: BRK-SOT-23-6, BSK-MSOP-8-3x3-P0.65, BRK-VSSOP-8-2.4x2.1-P0.5
Parts:
- J1, J2: value Conn_01x03 -> Conn_01x04; footprint Connector_PinHeader_2.54mm:PinHeader_1x03_P2.54mm_Vertical -> Connector_PinHeader_2.54mm:PinHeader_1x04_P2.54mm_Vertical; symbol Connector_Generic:Conn_01x03 -> Connector_Generic:Conn_01x04
- U1: value SC-70-6 -> VSSOP-8-2.4x2.1-P0.5; footprint Package_TO_SOT_SMD:SOT-363_SC-70-6_Handsoldering -> Package_SO:VSSOP-8_2.4x2.1mm_P0.5mm; symbol Connector_Generic:Conn_02x03_Counter_Clockwise -> Connector_Generic:Conn_02x04_Counter_Clockwise
Connections:
- wire segments 6 -> 8
Changed lines of the file:
@@
 EESchema Schematic File Version 4
-LIBS:BRK-SC-70-6-cache
+LIBS:BRK-VSSOP-8-2.4x2.1-P0.5-cache
 EELAYER 26 0
 EELAYER END
@@
 encoding utf-8
 Sheet 1 1
-Title "BRK-SC-70-6"
+Title "BRK-VSSOP-8-2.4x2.1-P0.5"
 Date ""
 Rev "v1.0"
@@
 $EndDescr
 $Comp
-L Connector_Generic:Conn_02x03_Counter_Clockwise U1
+L Connector_Generic:Conn_02x04_Counter_Clockwise U1
 U 1 1 5BD4B043
 P 5700 3900
 F 0 "U1" H 5750 4217 50  0000 C CNN
-F 1 "SC-70-6" H 5750 4126 50  0000 C CNN
-F 2 "Package_TO_SOT_SMD:SOT-363_SC-70-6_Handsoldering" H 5700 3900 50  0001 C CNN
+F 1 "VSSOP-8-2.4x2.1-P0.5" H 5750 4126 50  0000 C CNN
+F 2 "Package_SO:VSSOP-8_2.4x2.1mm_P0.5mm" H 5700 3900 50  0001 C CNN
 F 3 "~" H 5700 3900 50  0001 C CNN
 	1    5700 3900
@@
 $EndComp
 $Comp
-L Connector_Generic:Conn_01x03 J1
+L Connector_Generic:Conn_01x04 J1
 U 1 1 5BD4B0A3
 P 4800 3900
 F 0 "J1" H 4720 4217 50  0000 C CNN
-F 1 "Conn_01x03" H 4720 4126 50  0000 C CNN
-F 2 "Connector_PinHeader_2.54mm:PinHeader_1x03_P2.54mm_Vertical" H 4800 3900 50  0001 C CNN
+F 1 "Conn_01x04" H 4720 4126 50  0000 C CNN
+F 2 "Connector_PinHeader_2.54mm:PinHeader_1x04_P2.54mm_Vertical" H 4800 3900 50  0001 C CNN
 F 3 "~" H 4800 3900 50  0001 C CNN
 	1    4800 3900
@@
 $EndComp
 $Comp
-L Connector_Generic:Conn_01x03 J2
+L Connector_Generic:Conn_01x04 J2
 U 1 1 5BD4B172
-P 6700 3900
+P 6700 4000
 F 0 "J2" H 6619 3575 50  0000 C CNN
-F 1 "Conn_01x03" H 6619 3666 50  0000 C CNN
-F 2 "Connector_PinHeader_2.54mm:PinHeader_1x03_P2.54mm_Vertical" H 6700 3900 50  0001 C CNN
-F 3 "~" H 6700 3900 50  0001 C CNN
-	1    6700 3900
+F 1 "Conn_01x04" H 6619 3666 50  0000 C CNN
+F 2 "Connector_PinHeader_2.54mm:PinHeader_1x04_P2.54mm_Vertical" H 6700 4000 50  0001 C CNN
+F 3 "~" H 6700 4000 50  0001 C CNN
+	1    6700 4000
 	1    0    0    1
 $EndComp
@@
 Wire Wire Line
 	6500 4000 6000 4000
+Wire Wire Line
+	6000 4100 6500 4100
+Wire Wire Line
+	5500 4100 5000 4100
 $EndSCHEMATC
